File: circuits/telescope_circuit.brd (EAGLE design)
At the start: 53.6 x 68.6 mm, 22 parts, among them IC2 7805TV, J2 POWER_JACKSLT, U2 ATMEGA328P_PDIP_EZ, Y1 16MHz

Commit message: small fixes to the eagle pcb
Parts:
- removed J2: POWER_JACKSLT, SparkFun-Connectors:POWER_JACK_SLOT
- removed ON/OFF_BUTTON: (no value), con-amp-quick:02P
- added J1: POWER_JACKSLT, SparkFun-Connectors:POWER_JACK_SLOT
- added X1: (no value), con-ptr500:AK500/2
- R5: value 470 -> 330
- U2: value ATMEGA328P_PDIP_EZ -> 328P; device SparkFun-IC-Microcontroller:DIP28-SIMON-KIT -> SparkFun-IC-Microcontroller:DIP28
- moved BLUETOOTH 9.67 mm to (5.08, 47.0)
- moved IC2 7.62 mm to (2.54, 31.8)
Connections:
- net GND: now also J1.GND@1, J1.GND@2; no longer J2.GND@1, J2.GND@2
- net N$10: now also X1.1; no longer ON/OFF_BUTTON.2
- net VCC: now also J1.PWR, X1.2; no longer J2.PWR, ON/OFF_BUTTON.1
Routing:
- net N$8: track 139.3 -> 146.3 mm
- net VCC: track 17.3 -> 20.8 mm
- net N$5: track 12.2 -> 15.4 mm
- net N$10: track 82.5 -> 83.4 mm
- net N$6: track 12.7 -> 13.4 mm
