File: circuits/telescope_circuit.sch (EAGLE design)
At the start: 22 parts, among them IC2 7805TV, J2 POWER_JACKSLT, U2 ATMEGA328P_PDIP_EZ, Y1 16MHz

Commit message: small fixes to the eagle pcb
Parts:
- removed ON/OFF_BUTTON: (no value), con-amp-quick:M02
- added X1: (no value), con-ptr500:AK500/2
- R5: value 470 -> 330
- U2: value ATMEGA328P_PDIP_EZ -> 328P; device SparkFun-IC-Microcontroller:ATMEGA328P_PDIP_EZ -> SparkFun-IC-Microcontroller:ATMEGA328P_PDIP
- renumbered J2 to J1
Connections:
- net N$10: now also X1-1.KL; no longer ON/OFF_BUTTON.2
- net VCC: now also X1-2.KL; no longer ON/OFF_BUTTON.1
Changed lines of the file:
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@@
 </classes>
 <parts>
-<part name="U2" library="SparkFun-IC-Microcontroller" library_urn="urn:adsk.eagle:library:525" deviceset="ATMEGA328P_PDIP_EZ" device="" package3d_urn="urn:adsk.eagle:package:38949/1"/>
+<part name="U2" library="SparkFun-IC-Microcontroller" library_urn="urn:adsk.eagle:library:525" deviceset="ATMEGA328P_PDIP" device="" package3d_urn="urn:adsk.eagle:package:38942/1" value="328P"/>
 <part name="C1" library="SparkFun-Capacitors" library_urn="urn:adsk.eagle:library:510" deviceset="22PF" device="-PTH-2.54MM-200V-5%" package3d_urn="urn:adsk.eagle:package:37435/1" value="22pF"/>
 <part name="C2" library="SparkFun-Capacitors" library_urn="urn:adsk.eagle:library:510" deviceset="22PF" device="-PTH-2.54MM-200V-5%" package3d_urn="urn:adsk.eagle:package:37435/1" value="22pF"/>
@@
 <part name="R4" library="SparkFun-Resistors" deviceset="RESISTOR" device="AXIAL-0.3" value="10K"/>
 <part name="S2" library="switch-omron" library_urn="urn:adsk.eagle:library:377" deviceset="10-XX" device="" package3d_urn="urn:adsk.eagle:package:27496/1"/>
-<part name="R5" library="SparkFun-Resistors" deviceset="RESISTOR" device="AXIAL-0.3" value="470"/>
+<part name="R5" library="SparkFun-Resistors" deviceset="RESISTOR" device="AXIAL-0.3" value="330"/>
 <part name="LED1" library="led" library_urn="urn:adsk.eagle:library:259" deviceset="TLLY4400" device="" package3d_urn="urn:adsk.eagle:package:15797/1"/>
-<part name="J2" library="SparkFun-Connectors" deviceset="POWER_JACK" device="SLT"/>
 <part name="GND1" library="SparkFun-PowerSymbols" deviceset="GND" device=""/>
 <part name="R1" library="SparkFun-Resistors" deviceset="RESISTOR" device="AXIAL-0.3" value="3.3K"/>
@@
 <part name="C4" library="rcl" library_urn="urn:adsk.eagle:library:334" deviceset="CPOL-EU" device="E2.5-6" package3d_urn="urn:adsk.eagle:package:23349/1" value="100uF"/>
 <part name="SUPPLY1" library="SparkFun-PowerSymbols" deviceset="VCC" device=""/>
-<part name="ON/OFF_BUTTON" library="con-amp-quick" library_urn="urn:adsk.eagle:library:125" deviceset="M02" device="" package3d_urn="urn:adsk.eagle:package:5956/1"/>
 <part name="GND2" library="SparkFun-PowerSymbols" deviceset="GND" device=""/>
+<part name="J1" library="SparkFun-Connectors" library_urn="urn:adsk.eagle:library:513" deviceset="POWER_JACK" device="SLT" package3d_urn="urn:adsk.eagle:package:38222/1"/>
+<part name="X1" library="con-ptr500" library_urn="urn:adsk.eagle:library:181" deviceset="AK500/2" device="" package3d_urn="urn:adsk.eagle:package:9880/1"/>
 </parts>
 <sheets>
@@
 <attribute name="VALUE" x="4.572" y="28.575" size="1.778" layer="96" rot="R180"/>
 </instance>
-<instance part="J2" gate="G$1" x="-12.7" y="10.16" smashed="yes" rot="R90">
-<attribute name="VALUE" x="-22.86" y="5.08" size="1.778" layer="96" font="vector" rot="R90"/>
-<attribute name="NAME" x="-12.7" y="0" size="1.778" layer="95" font="vector" rot="R90"/>
-</instance>
 <instance part="GND1" gate="1" x="25.4" y="-2.54" smashed="yes">
 <attribute name="VALUE" x="25.4" y="-5.334" size="1.778" layer="96" align="top-center"/>
@@
 <attribute name="VALUE" x="-28.194" y="15.24" size="1.778" layer="96" rot="R90" align="bottom-center"/>
 </instance>
-<instance part="ON/OFF_BUTTON" gate="G$1" x="-27.94" y="25.4" smashed="yes">
-<attribute name="VALUE" x="-30.48" y="20.32" size="1.778" layer="96"/>
-<attribute name="NAME" x="-30.48" y="31.242" size="1.778" layer="95"/>
-</instance>
 <instance part="GND2" gate="1" x="162.56" y="22.86" smashed="yes">
 <attribute name="VALUE" x="162.56" y="20.066" size="1.778" layer="96" align="top-center"/>
+</instance>
+<instance part="J1" gate="G$1" x="-12.7" y="10.16" smashed="yes" rot="R90">
+<attribute name="VALUE" x="-22.86" y="0" size="1.778" layer="96" font="vector" rot="R90"/>
+<attribute name="NAME" x="-12.7" y="0" size="1.778" layer="95" font="vector" rot="R90"/>
+</instance>
+<instance part="X1" gate="-1" x="-25.4" y="30.48" smashed="yes">
+<attribute name="NAME" x="-26.67" y="31.369" size="1.778" layer="95" rot="R180"/>
+</instance>
+<instance part="X1" gate="-2" x="-25.4" y="25.4" smashed="yes">
+<attribute name="NAME" x="-26.67" y="26.289" size="1.778" layer="95" rot="R180"/>
+<attribute name="VALUE" x="-29.21" y="21.717" size="1.778" layer="96"/>
 </instance>
 </instances>
@@
 <pinref part="C2" gate="G$1" pin="2"/>
 <junction x="27.94" y="50.8"/>
-<pinref part="J2" gate="G$1" pin="GNDBREAK"/>
-<pinref part="J2" gate="G$1" pin="GND"/>
-<wire x1="-17.78" y1="12.7" x2="-15.24" y2="12.7" width="0.1524" layer="91"/>
-<wire x1="-15.24" y1="12.7" x2="25.4" y2="12.7" width="0.1524" layer="91"/>
-<junction x="-15.24" y="12.7"/>
 <junction x="25.4" y="12.7"/>
 <pinref part="C6" gate="G$1" pin="-"/>
@@
 <wire x1="17.78" y1="76.2" x2="17.78" y2="58.42" width="0.1524" layer="91"/>
 <junction x="17.78" y="58.42"/>
+<wire x1="-15.24" y1="12.7" x2="25.4" y2="12.7" width="0.1524" layer="91"/>
+<pinref part="J1" gate="G$1" pin="GND"/>
+<pinref part="J1" gate="G$1" pin="GNDBREAK"/>
+<wire x1="-17.78" y1="12.7" x2="-15.24" y2="12.7" width="0.1524" layer="91"/>
+<junction x="-15.24" y="12.7"/>
 </segment>
 <segment>
@@
 <wire x1="-7.62" y1="22.86" x2="-15.24" y2="22.86" width="0.1524" layer="91"/>
 <wire x1="-15.24" y1="48.26" x2="-15.24" y2="45.72" width="0.1524" layer="91"/>
-<wire x1="-15.24" y1="45.72" x2="-15.24" y2="27.94" width="0.1524" layer="91"/>
+<wire x1="-15.24" y1="45.72" x2="-15.24" y2="30.48" width="0.1524" layer="91"/>
 <pinref part="C6" gate="G$1" pin="+"/>
-<wire x1="-15.24" y1="27.94" x2="-15.24" y2="22.86" width="0.1524" layer="91"/>
+<wire x1="-15.24" y1="30.48" x2="-15.24" y2="22.86" width="0.1524" layer="91"/>
 <wire x1="-5.08" y1="45.72" x2="-15.24" y2="45.72" width="0.1524" layer="91"/>
 <junction x="-15.24" y="45.72"/>
@@
 <wire x1="157.48" y1="58.42" x2="172.72" y2="58.42" width="0.1524" layer="91"/>
 <junction x="172.72" y="58.42"/>
-<pinref part="ON/OFF_BUTTON" gate="G$1" pin="2"/>
-<wire x1="-20.32" y1="27.94" x2="-15.24" y2="27.94" width="0.1524" layer="91"/>
-<junction x="-15.24" y="27.94"/>
+<wire x1="-20.32" y1="30.48" x2="-15.24" y2="30.48" width="0.1524" layer="91"/>
+<junction x="-15.24" y="30.48"/>
 <wire x1="175.26" y1="88.9" x2="175.26" y2="68.58" width="0.1524" layer="91"/>
 <wire x1="175.26" y1="68.58" x2="180.34" y2="68.58" width="0.1524" layer="91"/>
@@
 <wire x1="172.72" y1="60.96" x2="180.34" y2="60.96" width="0.1524" layer="91"/>
 <wire x1="180.34" y1="60.96" x2="180.34" y2="63.5" width="0.1524" layer="91"/>
+<pinref part="X1" gate="-1" pin="KL"/>
 </segment>
 </net>
@@
 <pinref part="SUPPLY1" gate="G$1" pin="VCC"/>
 <wire x1="-27.94" y1="17.78" x2="-20.32" y2="17.78" width="0.1524" layer="91"/>
-<pinref part="J2" gate="G$1" pin="PWR"/>
-<pinref part="ON/OFF_BUTTON" gate="G$1" pin="1"/>
 <wire x1="-20.32" y1="12.7" x2="-20.32" y2="17.78" width="0.1524" layer="91"/>
 <wire x1="-20.32" y1="17.78" x2="-20.32" y2="25.4" width="0.1524" layer="91"/>
 <junction x="-20.32" y="17.78"/>
-</segment>
-</net>
+<pinref part="X1" gate="-2" pin="KL"/>
+<pinref part="J1" gate="G$1" pin="PWR"/>
+</segment>
+</net>
